File: Power-Primary.kicad_pcb (KiCad board)
At the start: 2 copper layers, 224.5 x 71.5 mm, 75 parts, among them J1 HV in, J10 SPARE, J11 SPARE, J12 SPARE, J13 SPARE, J14 SPARE, J15 SPARE, J16 SPARE, J17 SPARE, J2 Dashboard, J3 Telemetry, J4 Motor, J5 MPPT 1, J6 MPPT 2, J7 BPS, J8 Primary Disconn., J9 SPARE, U1 Mean_Well_12V

Commit message: Changes DC DC Converter to one that has more power
Parts:
- U1: footprint UTSVT_Power:Mean_Well_12V -> UTSVT_Power:RSD-150
- moved U1 96.1 mm to (130.1, 93.6)
- moved R18 44.1 mm to (218.1, 98.7)
- moved D17 44.1 mm to (213.4, 93.6)
- moved J12 29.3 mm to (164.9, 130.1)
- moved J13 29.3 mm to (180.1, 130.1)
- moved J14 29.3 mm to (195.4, 130.1)
- moved D11 29.3 mm to (173.8, 112.0)
- moved D12 29.3 mm to (189.0, 112.0)
- moved D13 29.3 mm to (204.3, 112.0)
- moved F12 29.3 mm to (168.3, 112.4)
- moved F13 29.3 mm to (183.1, 112.4)
- moved F14 29.3 mm to (198.3, 112.4)
- moved R11 29.3 mm to (173.8, 122.1)
- moved R12 29.3 mm to (189.0, 122.1)
- moved R13 29.3 mm to (204.3, 122.1)
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Routing:
- net Net-(F1-Pad2): track 60.7 -> 45.3 mm
- net /DC+: track 7.87 -> 21.3 mm
- net Net-(F1-Pad1): track 10.8 -> 18.5 mm
- net Net-(J1-Pad1): track 45.6 -> 40.6 mm
Other:
- board size 224.5 x 71.5 mm -> 244 x 92 mm
