File: Power-Primary.sch (KiCad schematic (older format))
At the start: 75 parts, among them J1 HV in, J10 SPARE, J11 SPARE, J12 SPARE, J13 SPARE, J14 SPARE, J15 SPARE, J16 SPARE, J17 SPARE, J2 Dashboard, J3 Telemetry, J4 Motor, J5 MPPT 1, J6 MPPT 2, J7 BPS, J8 Primary Disconn., J9 SPARE, U1 Mean_Well_12V

Commit message: Changes DC DC Converter to one that has more power
Parts:
- U1: footprint UTSVT_Power:Mean_Well_12V -> UTSVT_Power:RSD-150
Changed lines of the file:
@@
 F 0 "U1" H 3750 8787 60  0000 C CNN
 F 1 "Mean_Well_12V" H 3750 8681 60  0000 C CNN
-F 2 "UTSVT_Power:Mean_Well_12V" H 2900 7000 60  0001 C CNN
+F 2 "UTSVT_Power:RSD-150" H 2900 7000 60  0001 C CNN
 F 3 "" H 2900 7000 60  0001 C CNN
 	1    2900 7000
